File: schematic/agc.kicad_sch (KiCad schematic)
At the start: 72 parts, among them Q11 2N3904, Q8 2N3904, Q9 2N3904, U10 L78L33, U9 LM358

Commit message: Add PA schematic + some minor changes
Parts:
- L10, L11, L9: value L_Ferrite_Coupled_1423 -> FT37-43
Changed lines of the file:
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@@
       (effects (font (size 1.27 1.27)) (justify left))
     )
-    (property "Value" "L_Ferrite_Coupled_1423" (at 149.225 44.196 90)
+    (property "Value" "FT37-43" (at 149.225 44.196 90)
       (effects (font (size 1.27 1.27)) (justify left) hide)
     )
@@
       (effects (font (size 1.27 1.27)) (justify left))
     )
-    (property "Value" "L_Ferrite_Coupled_1423" (at 85.725 44.196 90)
+    (property "Value" "FT37-43" (at 85.725 44.196 90)
       (effects (font (size 1.27 1.27)) (justify left) hide)
     )
@@
       (effects (font (size 1.27 1.27)) (justify left))
     )
-    (property "Value" "L_Ferrite_Coupled_1423" (at 212.09 44.196 90)
+    (property "Value" "FT37-43" (at 212.09 44.196 90)
       (effects (font (size 1.27 1.27)) (justify left) hide)
     )

Commit message: Schematic: minor fixes
Other:
- note added: "10T bifilar @ FT37-43"
- note removed: "10T bifilar @ T37-43"
Changed lines of the file:
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@@
     (effects (font (size 1.27 1.27)) (justify left bottom))
   )
-  (text "10T bifilar\n@ T37-43" (at 210.185 59.055 0)
+  (text "10T bifilar\n@ FT37-43" (at 210.185 59.055 0)
     (effects (font (size 1.27 1.27)) (justify left bottom))
   )
@@
     (effects (font (size 1.27 1.27)) (justify left bottom))
   )
-  (text "10T bifilar\n@ T37-43" (at 147.32 59.055 0)
+  (text "10T bifilar\n@ FT37-43" (at 147.32 59.055 0)
     (effects (font (size 1.27 1.27)) (justify left bottom))
   )
-  (text "10T bifilar\n@ T37-43" (at 83.82 59.055 0)
+  (text "10T bifilar\n@ FT37-43" (at 83.82 59.055 0)
     (effects (font (size 1.27 1.27)) (justify left bottom))
   )
