File: schematic/bpfs.kicad_sch (KiCad schematic)
At the start: 54 parts

Commit message: Minor changes
Parts:
- renumbered L12 to L16, L12 to L17, L12 to L18, L12 to L19, L12 to L20, L12 to L21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
