File: schematic/power-amplifier.kicad_sch (KiCad schematic)
At the start: 55 parts, among them Q18 KT3142A, Q25 RD15HVF1, Q26 RD15HVF1, T1 FT37-43, T2 FT37-43, U18 LM7805

Commit message: Schematic: minor fixes
Parts:
- L33, L34: value 10T @ FT37-43 -> FT37-43
Other:
- note added: "10T @ FT37-43"
- note added: "w/ large heatsink"
Changed lines of the file:
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@@
+    (stroke (width 0) (type default))
+  )
+  (wire (pts (xy 64.135 133.985) (xy 67.31 133.985))
     (stroke (width 0) (type default))
   )
@@
     (stroke (width 0) (type default))
   )
-  (wire (pts (xy 65.405 148.59) (xy 67.31 148.59))
-    (stroke (width 0) (type default))
-  )
   (wire (pts (xy 234.95 100.965) (xy 237.49 100.965))
     (stroke (width 0) (type default))
@@
     (stroke (width 0) (type default))
   )
+  (wire (pts (xy 67.31 133.985) (xy 67.31 140.97))
+    (stroke (width 0) (type default))
+  )
   (wire (pts (xy 119.38 96.52) (xy 139.065 96.52))
     (stroke (width 0) (type default))
@@
     (stroke (width 0) (type default))
   )
-  (wire (pts (xy 67.31 148.59) (xy 67.31 140.97))
-    (stroke (width 0) (type default))
-  )
   (wire (pts (xy 237.49 96.52) (xy 237.49 100.965))
     (stroke (width 0) (type default))
@@
   (wire (pts (xy 55.88 168.275) (xy 57.15 168.275))
     (stroke (width 0) (type default))
+  )
+  (text "w/ large heatsink" (at 241.3 68.58 0)
+    (effects (font (size 1.27 1.27)) (justify left bottom))
   )
   (text "RX path, PA bypass" (at 58.42 161.925 0)
@@
   )
   (text "see /BPF Relays/" (at 17.78 163.195 0)
+    (effects (font (size 1.27 1.27)) (justify left bottom))
+  )
+  (text "w/ large heatsink" (at 241.3 118.11 0)
+    (effects (font (size 1.27 1.27)) (justify left bottom))
+  )
+  (text "10T @ FT37-43" (at 240.03 45.72 0)
     (effects (font (size 1.27 1.27)) (justify left bottom))
   )
@@
     (effects (font (size 1.27 1.27)) (justify left bottom))
   )
-  (text "TODO reference" (at 99.695 163.83 0)
+  (text "TODO reference" (at 99.695 163.195 0)
     (effects (font (size 1.27 1.27)) (justify left bottom))
   )
-  (text "10T bifilar\n@ FT50-43" (at 250.825 74.93 0)
+  (text "10T @ FT37-43" (at 240.03 95.885 0)
+    (effects (font (size 1.27 1.27)) (justify left bottom))
+  )
+  (text "10T bifilar\n@ FT50-43" (at 270.51 74.295 0)
     (effects (font (size 1.27 1.27)) (justify left bottom))
   )
@@
     )
   )
-  (global_label "TX_12V" (shape input) (at 65.405 148.59 180) (fields_autoplaced)
+  (global_label "TX_12V" (shape input) (at 64.135 133.985 180) (fields_autoplaced)
     (effects (font (size 1.27 1.27)) (justify right))
-    (property "Intersheetrefs" "${INTERSHEET_REFS}" (at 55.8469 148.59 0)
+    (property "Intersheetrefs" "${INTERSHEET_REFS}" (at 54.5769 133.985 0)
       (effects (font (size 1.27 1.27)) (justify right) hide)
     )
@@
       (effects (font (size 1.27 1.27)) (justify left))
     )
-    (property "Value" "10T @ FT37-43" (at 240.03 44.45 0)
-      (effects (font (size 1.27 1.27)) (justify left))
+    (property "Value" "FT37-43" (at 240.03 44.45 0)
+      (effects (font (size 1.27 1.27)) (justify left) hide)
     )
     (property "Footprint" "" (at 237.49 43.18 0)
@@
       (effects (font (size 1.27 1.27)) (justify left))
     )
-    (property "Value" "10T @ FT37-43" (at 240.03 93.98 0)
-      (effects (font (size 1.27 1.27)) (justify left))
+    (property "Value" "FT37-43" (at 240.03 93.98 0)
+      (effects (font (size 1.27 1.27)) (justify left) hide)
     )
     (property "Footprint" "" (at 237.49 92.71 0)

Commit message: Minor changes
Connections:
- net LPFS_IN renamed LPFS_OUT
Changed lines of the file:
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@@
     )
   )
-  (global_label "LPFS_IN" (shape output) (at 100.965 165.735 0) (fields_autoplaced)
+  (global_label "LPFS_OUT" (shape bidirectional) (at 100.965 165.735 0) (fields_autoplaced)
     (effects (font (size 1.27 1.27)) (justify left))
-    (property "Intersheetrefs" "${INTERSHEET_REFS}" (at 111.3699 165.735 0)
+    (property "Intersheetrefs" "${INTERSHEET_REFS}" (at 114.1745 165.735 0)
       (effects (font (size 1.27 1.27)) (justify left) hide)
     )

Commit message: Schematic: add relays to /LPFs/ sheet
Other:
- note added: "see /LPFs/"
- note removed: "TODO reference"
Changed lines of the file:
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@@
     (effects (font (size 1.27 1.27)) (justify left bottom))
   )
-  (text "see /BPF Relays/" (at 17.78 163.195 0)
+  (text "see /BPF Relays/" (at 17.78 163.83 0)
     (effects (font (size 1.27 1.27)) (justify left bottom))
   )
@@
     (effects (font (size 1.27 1.27)) (justify left bottom))
   )
-  (text "TODO reference" (at 99.695 163.195 0)
+  (text "see /LPFs/" (at 101.6 163.83 0)
     (effects (font (size 1.27 1.27)) (justify left bottom))
   )

Commit message: Minor changes
Parts:
- renumbered D22 to D23, D22 to D24, L12 to L35, Q18 to Q20, Q18 to Q21, Q18 to Q22, Q18 to Q23, Q18 to Q24, RL3 to RL27, RL3 to RL28
