File: schematic/rx.kicad_sch (KiCad schematic)
At the start: 34 parts, among them Q12 2N3904, U11 ADE-6

Commit message: Minor changes
Parts:
- renumbered C78 to C83, C79 to C84, C80 to C85, C81 to C86, C82 to C87, D14 to D15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
