File: schematic/tx-ssb.kicad_sch (KiCad schematic)
At the start: 37 parts, among them Q12 2N3904, U11 ADE-6, U15 NE5532

Commit message: Minor changes
Parts:
- renumbered C78 to C215, C79 to C216, C80 to C217, C81 to C218, C82 to C219, C212 to C220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
