File: pcbs/rxtx/agc.kicad_sch (KiCad schematic)
At the start: 79 parts, among them J6 Conn_01x02, Q1 MMBT3904, Q2 MMBT3904, Q3 MMBT3904, U1 L78L33, U2 LM358, U3 ADE-6

Commit message: Minor changes
Other:
- note added: "see /Root/"
- note removed: "see /Xtal Filters/"
Changed lines of the file:
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@@
     (effects (font (size 1.27 1.27)) (justify left bottom))
   )
-  (text "see /Xtal Filters/" (at 27.305 68.58 0)
+  (text "see /Root/" (at 29.845 68.58 0)
     (effects (font (size 1.27 1.27)) (justify left bottom))
   )
