File: pcbs/rxtx/rx.kicad_sch (KiCad schematic)
At the start: 36 parts, among them J7 Conn_01x02, J8 Conn_01x02, K7 G6K-2F-Y, K8 G6K-2F-Y, Q4 MMBT3904, Q5 MMBT3904, U4 ADE-6

Commit message: Minor changes
Other:
- note removed: "see /Xtal Filters/"
Changed lines of the file:
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@@
     (stroke (width 0) (type default))
   )
-  (text "see /Xtal Filters/" (at 254.635 62.23 0)
+  (text "see /Root/" (at 254.635 62.23 0)
     (effects (font (size 1.27 1.27)) (justify left bottom))
   )
