File: pcbs/rxtx/tx-common.kicad_sch (KiCad schematic)
At the start: 34 parts, among them J10 Conn_01x02, J9 Conn_01x02, K9 G6K-2F-Y, Q6 KT3142A, Q7 2N7002, Q8 MMBT3906, U5 ADE-6

Commit message: Minor changes
Other:
- note added: "see /Root/"
- note removed: "see /Xtal Filters/"
Changed lines of the file:
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@@
     (effects (font (size 1.27 1.27)) (justify left bottom))
   )
-  (text "see /Xtal Filters/" (at 67.31 144.78 0)
+  (text "see /Root/" (at 68.58 144.78 0)
     (effects (font (size 1.27 1.27)) (justify left bottom))
   )

Commit message: Various minor improvements
Parts:
- R52, R54: value 82 -> 51
- R53: value 82 -> 330
Other:
- note added: "22 dB attenuator"
- note added: "Anything between 12 dB and 22 dB will work. Less attenuation will give you more power in CW, however the power will be not even between the bands. See also .txDriveStrength in the firmware source code."
- note removed: "12 dB attenuator"
- moved on the sheet: J9, R52, R53, R54, U5

Commit message: Minor changes
Other:
- note added: "Anything between 12 dB and 22 dB will work. Less attenuation will give you more power in CW, however the power will not be even between the bands. See also .txDriveStrength in the firmware source code."
- note removed: "Anything between 12 dB and 22 dB will work. Less attenuation will give you more power in CW, however the power will be not even between the bands. See also .txDriveStrength in the firmware source code."
Changed lines of the file:
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@@
     (effects (font (size 1.27 1.27)) (justify left bottom))
   )
-  (text "Anything between 12 dB and 22 dB will work.\nLess attenuation will give you more power in CW,\nhowever the power will be not even between the bands.\nSee also .txDriveStrength in the firmware source code."
+  (text "Anything between 12 dB and 22 dB will work.\nLess attenuation will give you more power in CW,\nhowever the power will not be even between the bands.\nSee also .txDriveStrength in the firmware source code."
     (at 53.975 144.78 0)
     (effects (font (size 1.27 1.27)) (justify left bottom))
