File: pcbs/af/hbr-mk2-af.kicad_sch (KiCad schematic)
At the start: 36 parts, among them J1 Conn_01x02, J7 Conn_01x02, Q4 2N7002, Q5 2N7002, U1 LM7808, U4 NE5532

Commit message: AF PCB: fix typo
Other:
- note added: "Adjust to get a pure sine wave, about 0.7 Vpp"
- note removed: "Adjust to get a pure sine wave, about 7 Vpp"
Changed lines of the file:
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@@
     (stroke (width 0) (type default))
   )
-  (text "Adjust to get a pure \nsine wave, about 7 Vpp" (at 97.79 146.685 0)
+  (text "Adjust to get a pure \nsine wave, about 0.7 Vpp" (at 97.79 146.685 0)
     (effects (font (size 1.27 1.27)) (justify left bottom))
   )
