File: pcbs/af/af-amplifier.kicad_sch (KiCad schematic)
At the start: 63 parts, among them J2 Conn_01x02, J3 Conn_01x02, J4 Conn_01x03, J5 Conn_01x02, J6 Conn_01x03, Q1 MMBT3904, Q2 2N7002, Q3 2N7002, U2 NE5532, U3 TDA2003

Commit message: Minor changes
Other:
- note added: "see /Root/"
- note removed: "see /CW Tone/"
Changed lines of the file:
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@@
     (effects (font (size 1.27 1.27)) (justify left bottom))
   )
-  (text "see /CW Tone/" (at 160.655 99.06 0)
+  (text "see /Root/" (at 160.655 99.06 0)
     (effects (font (size 1.27 1.27)) (justify left bottom))
   )

Commit message: Minor changes
Parts:
- removed R14: DNP, symbol Device:R
Other:
- note removed: "In order to bypass mute circuit connect pins 3 of 2N7002s."
Changed lines of the file:
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@@
   (junction (at 52.07 150.495) (diameter 0) (color 0 0 0 0)
   )
-  (junction (at 102.235 66.04) (diameter 0) (color 0 0 0 0)
-  )
   (junction (at 229.87 76.835) (diameter 0) (color 0 0 0 0)
   )
@@
   (junction (at 131.445 127.635) (diameter 0) (color 0 0 0 0)
   )
-  (junction (at 154.305 66.04) (diameter 0) (color 0 0 0 0)
-  )
   (junction (at 145.415 127.635) (diameter 0) (color 0 0 0 0)
   )
@@
     (stroke (width 0) (type default))
   )
-  (wire (pts (xy 154.305 66.04) (xy 158.115 66.04))
+  (wire (pts (xy 145.415 66.04) (xy 158.115 66.04))
     (stroke (width 0) (type default))
   )
@@
     (stroke (width 0) (type default))
   )
-  (wire (pts (xy 145.415 66.04) (xy 154.305 66.04))
-    (stroke (width 0) (type default))
-  )
   (wire (pts (xy 131.445 127.635) (xy 131.445 140.97))
     (stroke (width 0) (type default))
@@
     (stroke (width 0) (type default))
   )
-  (wire (pts (xy 123.19 93.345) (xy 102.235 93.345))
-    (stroke (width 0) (type default))
-  )
   (wire (pts (xy 194.31 74.295) (xy 198.12 74.295))
     (stroke (width 0) (type default))
@@
     (stroke (width 0) (type default))
   )
-  (wire (pts (xy 130.81 93.345) (xy 154.305 93.345))
-    (stroke (width 0) (type default))
-  )
   (wire (pts (xy 127 66.04) (xy 127 70.485))
     (stroke (width 0) (type default))
@@
     (stroke (width 0) (type default))
   )
-  (wire (pts (xy 95.885 66.04) (xy 102.235 66.04))
-    (stroke (width 0) (type default))
-  )
   (wire (pts (xy 222.885 92.075) (xy 222.885 108.585))
     (stroke (width 0) (type default))
@@
     (stroke (width 0) (type default))
   )
-  (wire (pts (xy 102.235 93.345) (xy 102.235 66.04))
-    (stroke (width 0) (type default))
-  )
   (wire (pts (xy 208.28 51.435) (xy 203.2 51.435))
     (stroke (width 0) (type default))
@@
     (stroke (width 0) (type default))
   )
-  (wire (pts (xy 102.235 66.04) (xy 108.585 66.04))
+  (wire (pts (xy 95.885 66.04) (xy 108.585 66.04))
     (stroke (width 0) (type default))
   )
@@
   )
   (wire (pts (xy 107.315 140.97) (xy 107.315 130.175))
-    (stroke (width 0) (type default))
-  )
-  (wire (pts (xy 154.305 93.345) (xy 154.305 66.04))
     (stroke (width 0) (type default))
   )
@@
   )
   (text "VGND" (at 100.965 167.64 0)
-    (effects (font (size 1.27 1.27)) (justify left bottom))
-  )
-  (text "In order to bypass mute circuit\nconnect pins 3 of 2N7002s.\n"
-    (at 112.395 99.695 0)
     (effects (font (size 1.27 1.27)) (justify left bottom))
   )
@@
         )
       )
-    )
-  )
-  (symbol (lib_id "Device:R") (at 127 93.345 90) (unit 1)
-    (in_bom no) (on_board no) (dnp no) (fields_autoplaced)
-    (property "Reference" "R14" (at 127 87.63 90)
-      (effects (font (size 1.27 1.27)) hide)
-    )
-    (property "Value" "DNP" (at 127 90.17 90)
-      (effects (font (size 1.27 1.27)))
-    )
-    (property "Footprint" "" (at 127 95.123 90)
-      (effects (font (size 1.27 1.27)) hide)
-    )
-    (property "Datasheet" "~" (at 127 93.345 0)
-      (effects (font (size 1.27 1.27)) hide)
-    )
-    (pin "1")
-    (pin "2")
-    (instances
-      (project "hbr-mk2-af"
-        (path "/700c9878-4ed7-49d5-a273-77cf9d92989d/56e6206b-9eaf-48e3-8e65-5aed78d22a1d"
-          (reference "R14") (unit 1)
-        )
-      )
