File: pcbs/power/hbr-mk2-power.kicad_sch (KiCad schematic)
At the start: 42 parts, among them J1 Conn_01x08, J2 Conn_01x08, J3 Conn_01x08, J4 Conn_01x08, J5 Conn_01x03, Q1 2N7002, Q2 IRF4905, Q3 2N7002, Q4 IRF4905, Q5 IRF4905

Commit message: Minor changes
Other:
- note removed: "(was: ENABLE_RX_12V)"
Changed lines of the file:
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@@
     (stroke (width 0) (type default))
-  )
-  (text "(was: ENABLE_RX_12V)" (at 156.845 152.4 0)
-    (effects (font (size 1.27 1.27)) (justify left bottom))
-  )
-  (text "(was: ENABLE_RX_12V)" (at 140.97 36.195 0)
-    (effects (font (size 1.27 1.27)) (justify left bottom))
   )
   (global_label "RX_12V" (shape output) (at 266.065 99.695 0) (fields_autoplaced)
