File: pcbs/digital/hbr-mk2-digital.kicad_sch (KiCad schematic)
At the start: 98 parts, among them J1 Conn_01x09, J10 Conn_01x06, J11 Conn_01x05, J12 Conn_01x02, J13 Conn_01x02, J14 Conn_01x02, J2 Conn_01x02, J3 Conn_01x04, J4 Conn_01x04, J5 Conn_01x03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

Commit message: Minor changes
Other:
- note removed: "(was: ENABLE_RX_12V)"
Changed lines of the file:
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@@
     (effects (font (size 1.27 1.27)) (justify right bottom))
-  )
-  (text "(was: ENABLE_RX_12V)" (at 214.63 93.98 0)
-    (effects (font (size 1.27 1.27)) (justify left bottom))
   )
   (text "B8 & B9 are 5V-tolerant" (at 116.84 119.38 0)

Commit message: Various minor improvements
Parts:
- C3, C4, C7, C8: now left out of the parts list
- J6: value Conn_01x07 -> Si5351 Module
Changed lines of the file:
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@@
   )
   (symbol (lib_id "Device:C") (at 31.115 180.975 0) (unit 1)
-    (in_bom yes) (on_board yes) (dnp no) (fields_autoplaced)
+    (in_bom no) (on_board yes) (dnp no) (fields_autoplaced)
     (property "Reference" "C3" (at 34.925 179.705 0)
       (effects (font (size 1.27 1.27)) (justify left))
@@
       (effects (font (size 1.27 1.27)))
     )
-    (property "Value" "Conn_01x07" (at 74.93 160.655 0)
+    (property "Value" "Si5351 Module" (at 74.93 160.655 0)
       (effects (font (size 1.27 1.27)) hide)
     )
@@
   )
   (symbol (lib_id "Device:C") (at 41.91 140.97 0) (unit 1)
-    (in_bom yes) (on_board yes) (dnp no) (fields_autoplaced)
+    (in_bom no) (on_board yes) (dnp no) (fields_autoplaced)
     (property "Reference" "C8" (at 45.72 139.7 0)
       (effects (font (size 1.27 1.27)) (justify left))
@@
   )
   (symbol (lib_id "Device:C") (at 42.545 180.975 0) (unit 1)
-    (in_bom yes) (on_board yes) (dnp no) (fields_autoplaced)
+    (in_bom no) (on_board yes) (dnp no) (fields_autoplaced)
     (property "Reference" "C7" (at 46.355 179.705 0)
       (effects (font (size 1.27 1.27)) (justify left))
@@
   )
   (symbol (lib_id "Device:C") (at 29.845 140.97 0) (unit 1)
-    (in_bom yes) (on_board yes) (dnp no) (fields_autoplaced)
+    (in_bom no) (on_board yes) (dnp no) (fields_autoplaced)
     (property "Reference" "C4" (at 33.655 139.7 0)
       (effects (font (size 1.27 1.27)) (justify left))
