File: pcbs/pa/hbr-mk2-pa.kicad_sch (KiCad schematic)
At the start: 66 parts, among them J1 Conn_01x04, J2 Conn_01x02, J3 Conn_01x02, K1 G6K-2F-Y, K2 G6K-2F-Y, Q1 KT3142A, Q2 KT3142A, Q3 KT3142A, Q4 KT3142A, Q5 KT3142A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

Commit message: Minor changes
Other:
- note removed: "== General notes == - HFD4/12 relay is a full equivalent of G6K-2F-Y - KT3142A transistor is a full equvalent of 2N2369A - KT3142A can be replaced with another transistor with fT >= 500 Mhz"
Changed lines of the file:
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@@
-    (effects (font (size 1.27 1.27)) (justify left bottom))
-  )
-  (text "== General notes ==\n- HFD4/12 relay is a full equivalent of G6K-2F-Y\n- KT3142A transistor is a full equvalent of 2N2369A\n- KT3142A can be replaced with another transistor with fT >= 500 Mhz"
-    (at 210.82 27.94 0)
     (effects (font (size 1.27 1.27)) (justify left bottom))
   )

Commit message: Various minor improvements
Other:
- note added: "Quiescent currents: 50 mA per each RD15. Increase to 100 mA if you want a little more gain."
Changed lines of the file:
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@@
+    (effects (font (size 1.27 1.27)) (justify left bottom))
+  )
+  (text "Quiescent currents: 50 mA per each RD15.\nIncrease to 100 mA if you want a little more gain."
+    (at 187.96 141.605 0)
     (effects (font (size 1.27 1.27)) (justify left bottom))
   )
