File: pcbs/bfo/hbr-mk2-bfo.kicad_sch (KiCad schematic)
At the start: 40 parts, among them J1 Conn_01x02, J2 Conn_01x02, J3 Conn_01x02, K1 G6K-2F-Y, Q1 2N7002, Q2 MMBT3904, Q3 MMBT3904, Y1 DNP, Y2 9.000, Y3 9.000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

Commit message: Various minor improvements
Parts:
- C2, C4: value 30p -> 50p
- L1: value 18u -> 11u; now left out of the parts list
- L2: value 10u -> 0u; now left out of the parts list
- Y3: value 9.000 -> DNP; now left out of the parts list
Other:
- note added: "0u = jumper wire"
- note added: "11u = 53T @ T50-6"
- note added: "Some experimentation with different coils and crystals is required. Connecting two crystals in parralell sometimes allows to tune to the right frequency. Pay extra attention to the temperature stability of the generator."
- note added: "The signal level should be about 7 dBm, or 1.5 Vpp to the 50 Ohm load."
- note removed: "Some experimentation with different coils and crystals may be required."
Changed lines of the file:
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@@
     (effects (font (size 1.27 1.27)) (justify left bottom))
   )
-  (text "Some experimentation with different\ncoils and crystals may be required."
-    (at 103.505 167.005 0)
+  (text "The signal level should\nbe about 7 dBm, or 1.5 Vpp\nto the 50 Ohm load."
+    (at 254.635 135.89 0)
+    (effects (font (size 1.27 1.27)) (justify left bottom))
+  )
+  (text "Some experimentation with different\ncoils and crystals is required.\n\nConnecting two crystals in parralell\nsometimes allows to tune to the right\nfrequency.\n\nPay extra attention to the temperature\nstability of the generator."
+    (at 104.14 183.515 0)
     (effects (font (size 1.27 1.27)) (justify left bottom))
   )
@@
   )
   (text "Tuned to 9_000_633 Hz" (at 127.635 155.575 0)
+    (effects (font (size 1.27 1.27)) (justify left bottom))
+  )
+  (text "11u = 53T @ T50-6" (at 92.075 158.115 0)
+    (effects (font (size 1.27 1.27)) (justify left bottom))
+  )
+  (text "0u = jumper wire" (at 127.635 158.115 0)
     (effects (font (size 1.27 1.27)) (justify left bottom))
   )
@@
       (effects (font (size 1.27 1.27)) (justify left))
     )
-    (property "Value" "30p" (at 111.125 141.351 0)
+    (property "Value" "50p" (at 111.125 141.351 0)
       (effects (font (size 1.27 1.27)) (justify left))
     )
@@
   )
   (symbol (lib_id "Device:L") (at 107.95 116.205 0) (unit 1)
-    (in_bom yes) (on_board yes) (dnp no) (fields_autoplaced)
+    (in_bom no) (on_board yes) (dnp no) (fields_autoplaced)
     (property "Reference" "L1" (at 109.855 114.935 0)
       (effects (font (size 1.27 1.27)) (justify left))
     )
-    (property "Value" "18u" (at 109.855 117.475 0)
+    (property "Value" "11u" (at 109.855 117.475 0)
       (effects (font (size 1.27 1.27)) (justify left))
     )
@@
   )
   (symbol (lib_id "Device:Crystal") (at 125.73 128.27 90) (unit 1)
-    (in_bom yes) (on_board yes) (dnp no) (fields_autoplaced)
+    (in_bom no) (on_board yes) (dnp no) (fields_autoplaced)
     (property "Reference" "Y3" (at 130.175 127 90)
       (effects (font (size 1.27 1.27)) (justify right))
     )
-    (property "Value" "9.000" (at 130.175 129.54 90)
+    (property "Value" "DNP" (at 130.175 129.54 90)
       (effects (font (size 1.27 1.27)) (justify right))
     )
@@
       (effects (font (size 1.27 1.27)) (justify left))
     )
-    (property "Value" "30p" (at 135.89 141.986 0)
+    (property "Value" "50p" (at 135.89 141.986 0)
       (effects (font (size 1.27 1.27)) (justify left))
     )
@@
   )
   (symbol (lib_id "Device:L") (at 132.715 116.205 0) (unit 1)
-    (in_bom yes) (on_board yes) (dnp no) (fields_autoplaced)
+    (in_bom no) (on_board yes) (dnp no) (fields_autoplaced)
     (property "Reference" "L2" (at 134.62 114.935 0)
       (effects (font (size 1.27 1.27)) (justify left))
     )
-    (property "Value" "10u" (at 134.62 117.475 0)
-      (effects (font (size 1.27 1.27)) (justify left))
-    )
+    (property "Value" "0u" (at 134.62 117.475 0)
+      (effects (font (size 1.27 1.27)) (justify left))
+    )

Commit message: Minor changes
Other:
- note added: "The signal level should be about 7 dBm, or 1.5 Vpp into a 50 Ohm load."
- note removed: "The signal level should be about 7 dBm, or 1.5 Vpp to the 50 Ohm load."
Changed lines of the file:
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@@
     (effects (font (size 1.27 1.27)) (justify left bottom))
   )
-  (text "The signal level should\nbe about 7 dBm, or 1.5 Vpp\nto the 50 Ohm load."
+  (text "The signal level should\nbe about 7 dBm, or 1.5 Vpp\ninto a 50 Ohm load."
     (at 254.635 135.89 0)
     (effects (font (size 1.27 1.27)) (justify left bottom))
